File: pcb/matrix.kicad_sch (KiCad schematic)
At the start: 136 parts

Commit message: first pass at hotswap mechanical
Parts:
- removed D14, D60: 1N4148, Diode_SMD:D_SOD-123, symbol bakeneko-60-pcb-rescue:D-Device
- removed MX14, MX15: 1u, MX_Only:MXOnly-1U-NoLED, symbol bakeneko-60-pcb-rescue:SW_SPST-Switch
- removed MX58: 2.75u, MX_Only:MXOnly-2.75U-NoLED, symbol bakeneko-60-pcb-rescue:SW_SPST-Switch
- removed MX59, MX60, MX61, MX63, MX64, MX65, MX66: 1.25u, MX_Only:MXOnly-1.25U-NoLED, symbol bakeneko-60-pcb-rescue:SW_SPST-Switch
- removed MX62: 6.25u, MX_Only:MXOnly-6.25U-ReversedStabilizers-NoLED, symbol bakeneko-60-pcb-rescue:SW_SPST-Switch
- added H1: 2U Stab, Mounting_Keyboard_Stabilizer:Stabilizer_Cherry_MX_2.00u, symbol Mechanical:MountingHole
- added H2, H3: 2.25U Stab, Mounting_Keyboard_Stabilizer:Stabilizer_Cherry_MX_2.00u, symbol Mechanical:MountingHole
- added H4: 7U Stab, Mounting_Keyboard_Stabilizer:Stabilizer_Cherry_MX_7.00u, symbol Mechanical:MountingHole
- MX1, MX10, MX11, MX12, MX13, MX18, MX19, MX2, MX20, MX21, MX22, MX23, MX24, MX25, MX26, MX27, MX28, MX29, MX3, MX33, MX34, MX35, MX36, MX37, MX38, MX39, MX4, MX40, MX41, MX42, MX43, MX46, MX47, MX48, MX49, MX5, MX50, MX51, MX52, MX53, MX54, MX55, MX57, MX6, MX68, MX7, MX72, MX8, MX9: footprint MX_Only:MXOnly-1U-NoLED -> Switch_Keyboard_Hotswap_Kailh:SW_Hotswap_Kailh_MX_plated_1.00u
- MX16: footprint MX_Only:MXOnly-2U-NoLED -> Switch_Keyboard_Hotswap_Kailh:SW_Hotswap_Kailh_MX_plated_2.00u
- MX17, MX30, MX67, MX69, MX71, MX73: footprint MX_Only:MXOnly-1.5U-NoLED -> Switch_Keyboard_Hotswap_Kailh:SW_Hotswap_Kailh_MX_plated_1.50u
- MX31: footprint MX_Only:MXOnly-1.25U-NoLED -> Switch_Keyboard_Hotswap_Kailh:SW_Hotswap_Kailh_MX_plated_1.25u
- MX32, MX56: footprint MX_Only:MXOnly-1.75U-NoLED -> Switch_Keyboard_Hotswap_Kailh:SW_Hotswap_Kailh_MX_plated_1.75u
- MX44, MX45: footprint MX_Only:MXOnly-2.25U-NoLED -> Switch_Keyboard_Hotswap_Kailh:SW_Hotswap_Kailh_MX_plated_2.25u
- MX70: footprint MX_Only:MXOnly-7U-ReversedStabilizers-NoLED -> Switch_Keyboard_Hotswap_Kailh:SW_Hotswap_Kailh_MX_plated_7.00u
Other:
- moved on the sheet: MX16, MX67, MX68, MX69, MX70, MX71, MX72, MX73

Commit message: update bom
Parts:
- D1, D10, D11, D12, D13, D15, D16, D17, D18, D19, D2, D20, D21, D22, D23, D24, D25, D26, D27, D28, D29, D3, D30, D31, D32, D33, D34, D35, D36, D37, D38, D39, D4, D40, D41, D42, D43, D44, D45, D46, D47, D48, D49, D5, D50, D51, D52, D53, D54, D55, D56, D57, D58, D59, D6, D61, D62, D63, D7, D8, D9: LCSC (none) -> C81598; LCSC Part # C81598 -> (none)
- H1, H2, H3, H4: DNP (none) -> DNP
- MX1, MX10, MX11, MX12, MX13, MX16, MX17, MX18, MX19, MX2, MX20, MX21, MX22, MX23, MX24, MX25, MX26, MX27, MX28, MX29, MX3, MX30, MX31, MX32, MX33, MX34, MX35, MX36, MX37, MX38, MX39, MX4, MX40, MX41, MX42, MX43, MX44, MX45, MX46, MX47, MX48, MX49, MX5, MX50, MX51, MX52, MX53, MX54, MX55, MX56, MX57, MX6, MX67, MX68, MX69, MX7, MX70, MX71, MX72, MX73, MX8, MX9: LCSC (none) -> C2803348
