File: pcb/bakeneko-60-pcb.kicad_pcb (KiCad board)
At the start: 2 copper layers, 286.8 x 95.3 mm, 151 parts, among them J1 SM04B-SRSS-TB(LF)(SN), J2 AVR-ISP-6, SW1 Reset, U1 ATmega32U4-AU, U2 ATmega32U4-MU, Y1 16MHz

Commit message: first round off to fab for quote
Parts:
- added MX45: 2u, MX_Only:MXOnly-2U-NoLED, F.Cu at (335.5, 86.1)
- added MX58: 2.25u, MX_Only:MXOnly-2.25U-NoLED, F.Cu at (90.3, 143.2)
- moved D43 39.4 mm to (131.9, 144.0)
- moved D15 39.3 mm to (296.3, 86.8)
- moved D45 17.8 mm to (148.6, 144.0)
- moved D44 16.7 mm to (129.6, 144.0)
- moved D42 11.9 mm to (311.8, 125.0)
- moved D14 2.75 mm to (315.3, 86.8)
- moved D64 2.40 mm to (112.9, 144.0)
- moved D13 1.18 mm to (298.6, 86.8)
- moved D46 1.17 mm to (151.0, 144.0)
Routing:
- net Net-(D43-Pad2): track 16.4 -> 58.3 mm
- net Net-(D15-Pad2): track 7.01 -> 48.8 mm
- net ROW0: track 278.8 -> 256.9 mm
- net Net-(D42-Pad2): track 6.82 -> 18.8 mm
- net ROW2: track 269.4 -> 257.5 mm
- net COL14: track 307.3 -> 317.3 mm
- net Net-(D44-Pad2): track 5.93 -> 13.5 mm
- net Net-(D45-Pad2): track 6.82 -> 13.4 mm
- net COL0: track 117.3 -> 112.4 mm
- net Net-(D14-Pad2): track 5.29 -> 8.29 mm
- net Net-(D64-Pad2): track 13.5 -> 15.8 mm
- net ROW3: track 285.4 -> 284.0 mm
- net COL13: track 354.7 -> 355.8 mm
- net Net-(D13-Pad2): track 6.82 -> 5.83 mm
- net Net-(D46-Pad2): track 6.82 -> 5.87 mm
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Other:
- board size 286.8 x 95.3 mm -> 284.8 x 94.2 mm
- rule pad_to_mask_clearance: 0.05 -> 0
